Commit message: update obstacle avoiding with dynamic size

File: andy/obstacle_avoid/src/turtlebot3_description/urdf/1_depth_turtlebot3_burger.gazebo.xacro (robot description, xacro)
@@ -93,33 +93,43 @@
   </gazebo>
   <gazebo reference="base_scan">
-    <material>Gazebo/FlatBlack</material>
-    <sensor type="ray" name="lds_lfcd_sensor">
-      <pose>0 0 0 0 0 0</pose>
-      <visualize>$(arg laser_visual)</visualize>
-      <update_rate>5</update_rate>
-      <ray>
-        <scan>
-          <horizontal>
-            <samples>360</samples>
-            <resolution>1</resolution>
-            <min_angle>0.0</min_angle>
-            <max_angle>6.28319</max_angle>
-          </horizontal>
-        </scan>
-        <range>
-          <min>0.120</min>
-          <max>3.5</max>
-          <resolution>0.015</resolution>
-        </range>
-        <noise>
-          <type>gaussian</type>
-          <mean>0.0</mean>
-          <stddev>0.01</stddev>
-        </noise>
-      </ray>
-      <plugin name="gazebo_ros_lds_lfcd_controller" filename="libgazebo_ros_laser.so">
-        <topicName>scan</topicName>
-        <frameName>base_scan</frameName>
-      </plugin>
+    <sensor name="camera_depth(sensor)" type="depth">
+      <update_rate>20</update_rate>
+      <camera>
+        <horizontal_fov>1.5707813</horizontal_fov>
+        <image>
+          <width>640</width>
+          <height>480</height>
+          <format>R8G8B8</format>
+        </image>
+        <clip>
+          <near>0.5</near>
+          <far>5</far>
+        </clip>
+      </camera>
+        <plugin name="camera_depth_plugin" filename="libgazebo_ros_openni_kinect.so">
+          <baseline>0.2</baseline>
+          <alwaysOn>true</alwaysOn>
+          <!-- Keep this zero, update_rate in the parent <sensor> tag
+            will control the frame rate. -->
+          <updateRate>0.0</updateRate>
+          <cameraName>camera_depth</cameraName>
+          <imageTopicName>/depth_camera/image_raw</imageTopicName>
+          <cameraInfoTopicName>/depth_camera/camera_info</cameraInfoTopicName>
+          <depthImageTopicName>/depth_camera/depth_image</depthImageTopicName>
+          <depthImageInfoTopicName>/depth_camera/camera_info</depthImageInfoTopicName>
+          <pointCloudTopicName>/camera/depth/points</pointCloudTopicName>
+          <frameName>base_scan</frameName>
+          <baseline>0.12</baseline>
+          <!--hackBaseline>0.12</hackBaseline-->
+	  <distortionK1>0</distortionK1>
+          <distortionK2>0</distortionK2>
+          <distortionK3>0</distortionK3>
+          <distortionT1>0</distortionT1>
+          <distortionT2>0</distortionT2>
+          <CxPrime>0</CxPrime>
+          <Cx>0</Cx>
+          <Cy>0</Cy>
+          <focalLength>0</focalLength>
+        </plugin>
     </sensor>
   </gazebo>

File: andy/obstacle_avoid/src/turtlebot3_description/urdf/depth_turtlebot3_burger.gazebo.xacro (robot description, xacro)
@@ -96,16 +96,17 @@
       <update_rate>20</update_rate>
       <camera>
-        <horizontal_fov>1.047198</horizontal_fov>
+        <horizontal_fov>1.5707813</horizontal_fov>
         <image>
-          <width>64</width>
-          <height>48</height>
+          <width>640</width>
+          <height>480</height>
           <format>R8G8B8</format>
         </image>
         <clip>
           <near>0.05</near>
-          <far>3</far>
+          <far>5</far>
         </clip>
       </camera>
       <plugin name="camera_depth_plugin" filename="libgazebo_ros_depth_camera.so">
+	<baseline>0.12</baseline>
         <cameraName>camera_depth</cameraName>
         <alwaysOn>true</alwaysOn>
@@ -116,4 +117,13 @@
         <depthCameraInfoTopicName>depth_camera/depth_camera_info</depthCameraInfoTopicName>
         <frameName>base_scan</frameName>
+	<distortionK1>0</distortionK1>
+          <distortionK2>0</distortionK2>
+          <distortionK3>0</distortionK3>
+          <distortionT1>0</distortionT1>
+          <distortionT2>0</distortionT2>
+          <CxPrime>0</CxPrime>
+          <Cx>0</Cx>
+          <Cy>0</Cy>
+          <focalLength>0</focalLength>
       </plugin>
     </sensor>
